File: Hardware/SparkFun Refrigerator Gas Sensor (ZMOD4450).sch (EAGLE design)
At the start: 24 parts, among them J2 QWIIC_RIGHT_ANGLE, J4 QWIIC_RIGHT_ANGLE, U1 ZMOD4450 Refrigeration Gas Se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

Commit message: Checklist changes
Parts:
- removed LOGO2: SFE_LOGO_NAME_FLAME.1_INCH, SparkFun-Aesthetics:SFE_LOGO_NAME_FLAME.1_INCH
- renumbered JP1 to I2C
Other:
- note added: "7-bit unshifted I2C Address: 0x32"
- note added: "Vin: 1.7V-3.6V"
- note added: "ZMOD4450 Refrigeration Gas Sensor"
Changed lines of the file:
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@@
 <part name="R3" library="SparkFun-Resistors" deviceset="4.7KOHM" device="-0603-1/10W-1%" value="4.7k"/>
 <part name="SUPPLY1" library="SparkFun-PowerSymbols" deviceset="3.3V" device=""/>
-<part name="JP1" library="SparkFun-Jumpers" deviceset="JUMPER-SMT_3_2-NC_TRACE" device="_SILK" package3d_urn="urn:adsk.eagle:package:39289/1"/>
+<part name="I2C" library="SparkFun-Jumpers" deviceset="JUMPER-SMT_3_2-NC_TRACE" device="_SILK" package3d_urn="urn:adsk.eagle:package:39289/1"/>
 <part name="SUPPLY2" library="SparkFun-PowerSymbols" deviceset="3.3V" device=""/>
 <part name="SUPPLY4" library="SparkFun-PowerSymbols" deviceset="3.3V" device=""/>
@@
 <part name="FD4" library="SparkFun-Aesthetics" deviceset="FIDUCIAL" device="UFIDUCIAL"/>
 <part name="LOGO1" library="SparkFun-Aesthetics" deviceset="OSHW-LOGO" device="S"/>
-<part name="LOGO2" library="SparkFun-Aesthetics" deviceset="SFE_LOGO_NAME_FLAME" device=".1_INCH"/>
 <part name="J3" library="SparkFun-Connectors" deviceset="CONN_02" device="1X02_NO_SILK"/>
 </parts>
@@
 <text x="235.966" y="7.62" size="2.54" layer="94" font="vector">v01</text>
 <text x="41.148" y="126.746" size="1.778" layer="97" font="vector">Power</text>
-<text x="66.04" y="73.66" size="2.54" layer="97" font="vector" align="center">Connectors</text>
+<text x="2.54" y="81.28" size="2.54" layer="97" font="vector">Connectors</text>
 <text x="38.1" y="144.78" size="1.778" layer="97" font="vector">Cut the PWR
 jumper to disable
 the power LED</text>
 <wire x1="0" y1="86.36" x2="248.92" y2="86.36" width="0.1524" layer="97" style="longdash"/>
+<text x="2.54" y="180.34" size="2.54" layer="97" font="vector">ZMOD4450 Refrigeration Gas Sensor</text>
+<text x="2.54" y="177.8" size="1.778" layer="97" font="vector">Vin: 1.7V-3.6V</text>
+<text x="96.52" y="121.92" size="1.778" layer="97" font="vector">7-bit unshifted I2C Address: 0x32</text>
 </plain>
 <instances>
@@
 <attribute name="VALUE" x="104.14" y="155.194" size="1.778" layer="96" align="bottom-center"/>
 </instance>
-<instance part="JP1" gate="G$1" x="137.16" y="152.4" smashed="yes" rot="R270">
+<instance part="I2C" gate="G$1" x="137.16" y="152.4" smashed="yes" rot="R270">
 <attribute name="NAME" x="139.7" y="155.321" size="1.778" layer="95" font="vector"/>
 </instance>
@@
 <instance part="FD4" gate="G$1" x="236.22" y="27.94" smashed="yes"/>
 <instance part="LOGO1" gate="G$1" x="160.02" y="45.72" smashed="yes"/>
-<instance part="LOGO2" gate="G$1" x="182.88" y="38.1" smashed="yes"/>
 <instance part="J3" gate="G$1" x="88.9" y="43.18" smashed="yes" rot="MR0">
 <attribute name="VALUE" x="91.44" y="38.354" size="1.778" layer="96" font="vector" rot="MR0"/>
@@
 </segment>
 <segment>
-<pinref part="JP1" gate="G$1" pin="2"/>
+<pinref part="I2C" gate="G$1" pin="2"/>
 <pinref part="SUPPLY2" gate="G$1" pin="3.3V"/>
 <wire x1="137.16" y1="160.02" x2="137.16" y2="157.48" width="0.1524" layer="91"/>
@@
 <pinref part="R1" gate="G$1" pin="2"/>
 <wire x1="129.54" y1="149.86" x2="129.54" y2="152.4" width="0.1524" layer="91"/>
-<pinref part="JP1" gate="G$1" pin="3"/>
+<pinref part="I2C" gate="G$1" pin="3"/>
 <wire x1="129.54" y1="152.4" x2="132.08" y2="152.4" width="0.1524" layer="91"/>
 </segment>
@@
 <net name="N$3" class="0">
 <segment>
-<pinref part="JP1" gate="G$1" pin="1"/>
+<pinref part="I2C" gate="G$1" pin="1"/>
 <wire x1="142.24" y1="152.4" x2="144.78" y2="152.4" width="0.1524" layer="91"/>
 <pinref part="R2" gate="G$1" pin="2"/>

Commit message: Changing INT silk
Parts:
- added LOGO2: QWIIC_LOGO_5MM, SparkFun-Aesthetics:QWIIC_LOGO_5MM
Other:
- note added: "Cut the I2C jumper to remove the I2C pullups from the bus. Only do this if you have many devices on the bus and are seeing failures."
- note added: "x10"
- note removed: "v01"
Changed lines of the file:
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@@
 <part name="LOGO1" library="SparkFun-Aesthetics" deviceset="OSHW-LOGO" device="S"/>
 <part name="J3" library="SparkFun-Connectors" deviceset="CONN_02" device="1X02_NO_SILK"/>
+<part name="LOGO2" library="SparkFun-Aesthetics" deviceset="QWIIC_LOGO" device="_5MM"/>
 </parts>
 <sheets>
@@
 <plain>
 <text x="166.116" y="11.176" size="2.54" layer="94" font="vector">Andy England</text>
-<text x="235.966" y="7.62" size="2.54" layer="94" font="vector">v01</text>
+<text x="235.966" y="7.62" size="2.54" layer="94" font="vector">x10</text>
 <text x="41.148" y="126.746" size="1.778" layer="97" font="vector">Power</text>
 <text x="2.54" y="81.28" size="2.54" layer="97" font="vector">Connectors</text>
@@
 <text x="2.54" y="177.8" size="1.778" layer="97" font="vector">Vin: 1.7V-3.6V</text>
 <text x="96.52" y="121.92" size="1.778" layer="97" font="vector">7-bit unshifted I2C Address: 0x32</text>
+<text x="144.78" y="154.94" size="1.778" layer="97" font="vector">Cut the I2C jumper to remove the I2C
+pullups from the bus. Only do this if you
+have many devices on the bus and are
+seeing failures.</text>
 </plain>
 <instances>
@@
 <attribute name="NAME" x="91.44" y="48.768" size="1.778" layer="95" font="vector" rot="MR0"/>
 </instance>
+<instance part="LOGO2" gate="G$1" x="238.76" y="40.64" smashed="yes"/>
 </instances>
 <busses>
